Commit message: curent

File: src/ruka/config/ruka.ros2_control.xacro (robot description, xacro)
@@ -6,5 +6,5 @@
             <hardware>
                 <!-- By default, set up controllers for simulation. This won't work on real hardware -->
-                <plugin>joint_trajectory_controller/JointTrajectoryController</plugin>
+                <plugin>ruka/RukaSystem</plugin>
             </hardware>
             <joint name="base_link__link_01">

File: src/ruka/config/ruka.urdf (robot description, URDF)
Before this commit: robot ruka, 12 links, 11 joints
Joints:
- joint base_link__link_01: limit lower=-3.14 upper=3.14 effort=1000.0 velocity=0.5 -> lower=-2.96 upper=2.96 effort=1000.0 velocity=0.5
- joint link_01__link_02: limit lower=-3.14 upper=3.14 effort=1000.0 velocity=0.5 -> lower=-3.57 upper=0 effort=1000.0 velocity=0.5; origin xyz=0.01 0 0.179 rpy=1.57 0 0 -> xyz=0.01 0 0.179 rpy=1.57 -1.57 0
- joint link_02__link_03: limit lower=-3.14 upper=3.14 effort=1000.0 velocity=0.5 -> lower=0.035 upper=5.23 effort=1000.0 velocity=0.5; origin xyz=0 0.28 0 rpy=0 0 1.57 -> xyz=0 0.28 0 rpy=0 0 0.0175
- joint link_03__link_04: limit lower=-3.14 upper=3.14 effort=1000.0 velocity=0.5 -> lower=-2.87 upper=2.87 effort=1000.0 velocity=0.5
- joint link_04__link_05: limit lower=-3.14 upper=3.14 effort=1000.0 velocity=0.5 -> lower=-2.44 upper=2.44 effort=1000.0 velocity=0.5

File: src/ruka/config/ruka.urdf.xacro (robot description, xacro)
@@ -1,4 +1,5 @@
 <?xml version="1.0"?>
 <robot xmlns:xacro="http://www.ros.org/wiki/xacro" name="ruka">
+    <xacro:arg name="prefix" default="" />
     <xacro:arg name="initial_positions_file" default="initial_positions.yaml" />
     <!-- Import ruka urdf file -->
@@ -6,4 +7,14 @@
     <!-- Import control_xacro -->
     <xacro:include filename="$(find ruka)/config/ruka.ros2_control.xacro" />
-    <xacro:ruka_ros2_control name="ruka" initial_positions_file="$(arg initial_positions_file)"/>
+    <xacro:include filename="$(find ruka)/config/imu.ros2_control.xacro" />
+    <xacro:ruka_ros2_control name="RukaSystemController" initial_positions_file="$(arg initial_positions_file)"/>
+    <!--
+    <xacro:ruka_ros2_sensor
+     name="ruka" prefix="$(arg prefix)"
+     use_mock_hardware="$(arg use_mock_hardware)"
+     mock_sensor_commands="$(arg mock_sensor_commands)" />
+    -->
+    <xacro:ruka_ros2_sensor
+     name="RukaSensorSee" prefix="$(arg prefix)"
+      />
 </robot>
